File: Metronome.kicad_pcb (KiCad board)
At the start: 2 copper layers, 24.8 x 24.5 mm, 31 parts, among them CON1 PDI_50mil, IC1 ATXMEGA8E5-MU, P1 USB_B, Q1 Q_PMOS_GSD, U1 AS1117, U2 NCP706A, Y1 Crystal

Commit message: Update copyright on board
Other:
- board text added: "Micronome Rev. 1.0 © Kevin Ward 2016"
- board text removed: "Micronome Rev. 1.0 © Kevin Ward 2015"
Changed lines of the file:
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@@
     (pad "" thru_hole circle (at 0 0) (size 2 2) (drill 2) (layers *.Cu *.Mask F.SilkS))
   )
-  (gr_text "Micronome Rev. 1.0\n© Kevin Ward 2015" (at 68.9 74.4 90) (layer B.SilkS)
+  (gr_text "Micronome Rev. 1.0\n© Kevin Ward 2016" (at 68.9 74.4 90) (layer B.SilkS)
     (effects (font (size 0.8 0.8) (thickness 0.2)) (justify mirror))
   )
